Commit message: feat: upgraded sensor with rgb-d camera and created new launch file that runs RTAB-map.
For this commit, the my_robot package has been updated with a kinetic
sensor instead of a regular rgb camera. The urdfs have been modified
to make this update proper. A launch file specifically for mapping has
been created as well. The launch file will run the rtabmap node which
will also open up rtabmapviz. This node gives us greater visiblity to
feature mapping, loop closures, and etc.

File: my_robot/urdf/my_robot.xacro (robot description, xacro)
@@ -167,5 +167,5 @@
     <dynamics damping="1.0" friction="1.0"/>
   </joint>
-  <link name="camera">
+  <link name="camera_link">
     <inertial>
     <mass value="0.1"/>
@@ -194,7 +194,14 @@
     <origin xyz="0.2 0 0" rpy="0 0 0"/>
     <parent link="chassis"/>
-    <child link="camera"/>
-    <axis xyz="0 1 0" rpy="0 0 0"/>
-  </joint>
+    <child link="camera_link"/>
+    <axis xyz="0 1 0" rpy="0 0 0"/>
+  </joint>
+  <joint name="camera_optical_joint" type="fixed">
+    <origin xyz="0 0 0" rpy="-1.5707 0 -1.5707"/>
+    <parent link="camera_link"/>
+    <child link="camera_link_optical"/>
+  </joint>
+  <link name="camera_link_optical">
+  </link>
   <link name="hokuyo">
     <interial>
